File: 3 - ELECTRONIQUE & ELECTRIQUE/31 - TEST/LAMP_OUTDOOR_BATTERY/LAMP_OUTDOOR_BATTERY.kicad_sch (KiCad schematic)
At the start: 32 parts, among them J1 629722000214, J2 Batt+, J3 Batt-, SW1 SW_SPST, U1 MCP73833-FCI_UN, U2 MT3608, U3 AT42QT1012-MAHR

Commit message: Conception PCB suite
Parts:
- removed F1: Fuse_Small, Fuse:Fuse_1206_3216Metric_Pad1.42x1.75mm_HandSolder, symbol Device:Fuse_Small
- added C7: 0.1uF, Capacitor_SMD:C_0402_1005Metric_Pad0.74x0.62mm_HandSolder, symbol Device:C
- added J4: Led+, LAMP_OUTDOOR_BATTERY:BatteryPole, symbol Connector:Conn_01x01_Pin
- added J5: Led-, LAMP_OUTDOOR_BATTERY:BatteryPole, symbol Connector:Conn_01x01_Pin
- added J6: Electrode Sensor, LAMP_OUTDOOR_BATTERY:BatteryPole, symbol Connector:Conn_01x01_Pin
- added Q1, Q2: IRLML6344, Package_TO_SOT_SMD:SOT-23-3, symbol Transistor_FET:IRLML0030
- added R14: 2.2K, Resistor_SMD:R_0402_1005Metric_Pad0.72x0.64mm_HandSolder, symbol Device:R
- added R15: 330, Resistor_SMD:R_0402_1005Metric_Pad0.72x0.64mm_HandSolder, symbol Device:R
- added U4: BQ29737DSER, Package_SON:WSON-6_1.5x1.5mm_P0.5mm, symbol LAMP_OUTDOOR_BATTERY:BQ29737DSER
Connections:
- net Battery+ is gone; now on net +BATT: J2.1 (Pin_1)
- net +BATT: now also R15.1
- net ElecSensor: now also J6.1 (Pin_1)
- net GND: now also J5.1 (Pin_1), Q1.2 (S), R14.2; no longer J3.1 (Pin_1)
- net Led_V+: now also J4.1 (Pin_1)
- new net: C7.2, R15.2, U4.5 (BAT)
- new net: Q1.1 (G), U4.2 (COUT)
- new net: Q1.3 (D), Q2.3 (D)
- new net: R14.1, U4.6 (V-)
- new net: Q2.1 (G), U4.3 (DOUT)
- new net Battery-: C7.1, J3.1 (Pin_1), Q2.2 (S), U4.4 (VSS)
- no-connect marks 9 -> 10
Other:
- note added: "BQ29737DSER Circuit Protection charge/discharge"
- moved on the sheet: C1, C2, C3, C4, C5, C6, D1, D2, D3, D4, J1, J2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

Commit message: PCB & Conception 3D V1
Parts:
- L1: footprint Inductor_SMD:L_0805_2012Metric_Pad1.15x1.40mm_HandSolder -> LAMP_OUTDOOR_BATTERY:IND_F1C1-201608-4R7M
Connections:
- net +5V: no longer C6.2, U3.7 (VDD)
- net +BATT: now also C6.2, U3.7 (VDD)

Commit message: Commande composants
Parts:
- C5: value ~ -> 10nF
- R10: value ~ -> 10K
- R11: value ~ -> 1M
Other:
- note added: "C5 -> typical values 2.2nF to 50nF depending on the sensitivity required R10 -> limit ESD currents and suppress radio frequenxy interference (RFI), should be 4.7k to 33k R11 -> 1M ohms"
Changed lines of the file:
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@@
 		)
 	)
+	(text "C5 -> typical values 2.2nF to 50nF depending on the sensitivity required\nR10 -> limit ESD currents and suppress radio frequenxy interference (RFI), should be 4.7k to 33k\nR11 -> 1M ohms"
+		(exclude_from_sim no)
+		(at 61.214 146.304 0)
+		(effects
+			(font
+				(size 1 1)
+			)
+		)
+	)
 	(text "Convertisseur Boost 3.7V-5V"
 		(exclude_from_sim no)
@@
 			)
 		)
-		(property "Value" "~"
+		(property "Value" "1M"
 			(at 41.91 126.9999 0)
 			(effects
@@
 			)
 		)
-		(property "Value" "~"
+		(property "Value" "10K"
 			(at 41.91 109.2199 0)
 			(effects
@@
 			)
 		)
-		(property "Value" "~"
+		(property "Value" "10nF"
 			(at 45.974 115.57 0)
 			(effects
